File: electronics/stage4/monitoring-cell/channel0.kicad_sch (KiCad schematic)
At the start: 26 parts, among them J100 SOURCE 0 RETURN SHUNT, J101 SOURCE 0 DRIVER PERMISSION, U100 INA241A2IDR, U101 OPA391DBVR, U102 OPA391DBVR, U103 ADS8866IDGSR, U104 TLV3202IDR, U105 SN74LVC1G11DBVR, U106 SN74LVC1G74DCUR

Commit message: Verify phase-charge study and portable source reproduction
Parts:
- U101, U102: value OPA391DBVR -> OPA391DCKR; footprint ato_s4:SOT-23-5 -> ato_s4:SOT-353_SC-70-5
Connections:
- net CH0_ADC_BUF: now also U102.3 (IN-); no longer U102.1 (OUT)
- net CH0_Q_INT: now also U101.4 (OUT), U102.1 (IN+); no longer U101.1 (OUT), U102.3 (IN+)
- net CH0_SUM: now also U101.3 (IN-); no longer U101.4 (IN-)
- net V_MID: now also U101.1 (IN+); no longer U101.3 (IN+)
