File: electronics/stage4/monitoring-cell/channel1.kicad_sch (KiCad schematic)
At the start: 26 parts, among them J200 SOURCE 1 RETURN SHUNT, J201 SOURCE 1 DRIVER PERMISSION, U200 INA241A2IDR, U201 OPA391DBVR, U202 OPA391DBVR, U203 ADS8866IDGSR, U204 TLV3202IDR, U205 SN74LVC1G11DBVR, U206 SN74LVC1G74DCUR

Commit message: Verify phase-charge study and portable source reproduction
Parts:
- U201, U202: value OPA391DBVR -> OPA391DCKR; footprint ato_s4:SOT-23-5 -> ato_s4:SOT-353_SC-70-5
Connections:
- net CH1_ADC_BUF: now also U202.3 (IN-); no longer U202.1 (OUT)
- net CH1_Q_INT: now also U201.4 (OUT), U202.1 (IN+); no longer U201.1 (OUT), U202.3 (IN+)
- net CH1_SUM: now also U201.3 (IN-); no longer U201.4 (IN-)
- net V_MID: now also U201.1 (IN+); no longer U201.3 (IN+)
